File: KleverLogger.kicad_pcb (KiCad board)
At the start: 2 copper layers, 50 x 50 mm, 51 parts, among them J1 CAN, J5 USB_C_Receptacle_USB2.0, J7 RS485, U1 ESP32-C3-WROOM-02, U2 AP2112K-3.3, U3 TJA1051T-3, U5 MAX485E, U6 USBLC6-2SC6, U9 LM5164DDA

Commit message: After ordering v0.1
Parts:
- removed R18: 10k, Resistor_SMD:R_0805_2012Metric
- added C10: 100n, Capacitor_SMD:C_0805_2012Metric, B.Cu at (71.0, 91.9)
- added C11: 100n, Capacitor_SMD:C_0805_2012Metric, B.Cu at (80.7, 92.4)
- added C12: 10u, Capacitor_SMD:C_0805_2012Metric, B.Cu at (77.7, 107.0)
- added C13: 10u, Capacitor_SMD:C_0805_2012Metric, B.Cu at (80.8, 103.4)
- added C6: 100n, Capacitor_SMD:C_0805_2012Metric, B.Cu at (105.0, 109.0)
- added C7: 100n, Capacitor_SMD:C_0805_2012Metric, B.Cu at (105.0, 101.1)
- added C8: 100n, Capacitor_SMD:C_0805_2012Metric, F.Cu at (98.0, 119.5)
- added C9: 10u, Capacitor_SMD:C_0805_2012Metric, B.Cu at (71.0, 94.0)
- added D6: WS2812B, LED_SMD:LED_WS2812B_PLCC4_5.0x5.0mm_P3.2mm, F.Cu at (105.0, 95.0)
- added D7: WS2812B, LED_SMD:LED_WS2812B_PLCC4_5.0x5.0mm_P3.2mm, F.Cu at (105.0, 101.0)
- added D8: WS2812B, LED_SMD:LED_WS2812B_PLCC4_5.0x5.0mm_P3.2mm, F.Cu at (105.0, 107.0)
- added J2: BATTERY, Connector_JST:JST_PH_S2B-PH-K_1x02_P2.00mm_Horizontal, F.Cu at (65.0, 134.6)
- added SW1: SW_SPST, Fair:Flat_SMD_Switch, F.Cu at (67.2, 100.4)
- added TP1: 3V3, Fair:TestPoint_Pad_D0.8mm, F.Cu at (62.0, 98.1)
- added TP10: CANH, Fair:TestPoint_Pad_D0.8mm, F.Cu at (89.1, 130.2)
- added TP11: CANL, Fair:TestPoint_Pad_D0.8mm, F.Cu at (80.1, 130.4)
- added TP12: IO3, Fair:TestPoint_Pad_D0.8mm, F.Cu at (98.3, 94.1)
- added TP2: 5V, Fair:TestPoint_Pad_D0.8mm, F.Cu at (76.5, 106.5)
- added TP3: RX, Fair:TestPoint_Pad_D0.8mm, F.Cu at (90.0, 105.3)
- added TP4: DE, Fair:TestPoint_Pad_D0.8mm, F.Cu at (92.4, 106.3)
- added TP5: TX, Fair:TestPoint_Pad_D0.8mm, F.Cu at (96.2, 101.7)
- added TP6: MOSI, Fair:TestPoint_Pad_D0.8mm, F.Cu at (70.2, 92.2)
- added TP7: MISO, Fair:TestPoint_Pad_D0.8mm, F.Cu at (68.1, 97.4)
- added TP8: SCK, Fair:TestPoint_Pad_D0.8mm, F.Cu at (71.8, 95.8)
- added TP9: CS, Fair:TestPoint_Pad_D0.8mm, F.Cu at (72.6, 100.2)
- C1, C2: value 10uF/6.3V -> 100n
- C3: value 1uF/25V -> 100n
- C35, C36, C37, C50, C52, C53, R67, R83, R84, R85: moved to F.Cu
- D1: value Red -> ~; footprint LED_SMD:LED_0603_1608Metric -> LED_SMD:LED_0805_2012Metric
- D2, U4, U5: moved to B.Cu
- D3: value Blue -> 100V/3A; footprint LED_SMD:LED_0603_1608Metric -> Diode_SMD:D_SOD-123F
- D4: value Emerald -> 100V/3A; footprint LED_SMD:LED_0603_1608Metric -> Diode_SMD:D_SOD-123F; moved to B.Cu
- R17: value 10k -> 10
- R4: value 220 -> 10k
- R5, R7: value 1k -> 10k
- R6: value 10k -> 220
- moved R15 77.2 mm to (62.5, 101.5), turned to -90 degrees
- moved U4 67.8 mm to (68.5, 106.9), turned to 90 degrees
- moved R16 67.2 mm to (64.4, 101.5), turned to -90 degrees
- moved R14 66.2 mm to (63.0, 107.9), turned to 90 degrees
- moved C50 61.2 mm to (71.9, 119.0), turned to -90 degrees
- moved R2 58.9 mm to (80.7, 94.4)
- moved C5 58.7 mm to (69.8, 100.9), turned to 180 degrees
- moved R13 57.8 mm to (71.6, 97.5), turned to -90 degrees
- moved R4 55.4 mm to (64.6, 113.0)
- moved R1 50.3 mm to (84.1, 106.6), turned to -90 degrees
- moved C35 49.7 mm to (76.0, 119.0), turned to 90 degrees
- moved R12 49.0 mm to (91.0, 128.5), turned to -90 degrees
- moved R7 49.0 mm to (74.0, 109.0), turned to -90 degrees
- moved C1 48.7 mm to (80.3, 125.0), turned to 90 degrees
- moved C37 48.0 mm to (74.0, 123.0), turned to 90 degrees
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Connections:
- net /C3_RX renamed /RS485_RX
- net /C3_TX renamed /RS485_TX
- C3 pad 1: /EN/CHIP_PU -> +5V
- C50 pad 1: /BST -> /SW
- C50 pad 2: /SW -> /BST
- C52 pad 1: BAT+ -> /VIN
- D3 pad 1: GND -> /VIN
- D4 pad 1: GND -> +5V
- J1 pad 1: unconnected-(J1-Pin_1-Pad1) -> Net-(D4-A)
- J1 pad 2: unconnected-(J1-Pin_2-Pad2) -> /CANL
- J1 pad 3: unconnected-(J1-Pin_3-Pad3) -> /CANH
- J1 pad 4: unconnected-(J1-Pin_4-Pad4) -> GND
- J5 pad A4: Net-(U6-VBUS) -> /Vbus
- J5 pad A9: Net-(U6-VBUS) -> /Vbus
- J5 pad B4: Net-(U6-VBUS) -> /Vbus
- J5 pad B9: Net-(U6-VBUS) -> /Vbus
- R1 pad 1: Net-(D4-A) -> +3V3
- R1 pad 2: /LED_Green -> Net-(D1-A)
- R11 pad 2: Net-(D2-A2) -> Net-(D2-A1)
- R12 pad 2: Net-(D2-A1) -> Net-(D2-A2)
- R14 pad 1: /SD_CS -> +3V3
- R14 pad 2: +3V3 -> Net-(U4-DAT1)
- R15 pad 1: Net-(U4-DAT2) -> +3V3
- R15 pad 2: +3V3 -> /SD_MISO
- R16 pad 1: Net-(U4-DAT1) -> +3V3
- R16 pad 2: +3V3 -> /SD_MOSI
- R17 pad 1: /SD_MISO -> /GPIO3
- R17 pad 2: +3V3 -> Net-(D6-DIN)
- R3 pad 2: /LED_Green -> /GPIO2
- R4 pad 1: /CANL -> +3V3
- R4 pad 2: /CANH -> /SD_CS
- R5 pad 1: Net-(D3-A) -> +3V3
- R5 pad 2: /LED_Blue -> /GPIO8
- R6 pad 1: +3V3 -> /CANH
- R6 pad 2: /GPIO8 -> /CANL
- R7 pad 2: Net-(D1-A) -> Net-(U4-DAT2)
- U1 pad 10: unconnected-(U1-IO10-Pad10) -> /RS485_DE
- U1 pad 13: unconnected-(U1-IO18-Pad13) -> /USB_D-
- U1 pad 14: /C3_DE_RS485 -> /USB_D+
- U1 pad 15: unconnected-(U1-IO3-Pad15) -> /GPIO3
- U1 pad 16: /LED_Green -> /GPIO2
- U1 pad 17: unconnected-(U1-IO1-Pad17) -> /CAN_TX
- U1 pad 18: unconnected-(U1-IO0-Pad18) -> /CAN_RX
- U1 pad 3: unconnected-(U1-IO4-Pad3) -> /SD_MOSI
- U1 pad 4: unconnected-(U1-IO5-Pad4) -> /SD_SCK
- U1 pad 5: unconnected-(U1-IO6-Pad5) -> /SD_MISO
- U1 pad 6: unconnected-(U1-IO7-Pad6) -> /SD_CS
- U1 pad 8: unconnected-(U1-IO9-Pad8) -> Net-(SW1-A)
- U5 pad 2: /C3_DE_RS485 -> /RS485_DE
- U5 pad 3: /C3_DE_RS485 -> /RS485_DE
- U6 pad 1: unconnected-(U6-I/O1-Pad1) -> Net-(J5-D--PadA7)
- U6 pad 3: unconnected-(U6-I/O2-Pad3) -> Net-(J5-D+-PadA6)
- U6 pad 4: unconnected-(U6-I/O2-Pad4) -> /USB_D+
- U6 pad 5: Net-(U6-VBUS) -> +5V
- U6 pad 6: unconnected-(U6-I/O1-Pad6) -> /USB_D-
- U9 pad 2: BAT+ -> /VIN
- U9 pad 3: BAT+ -> /VIN
Routing:
- net +3V3: track 0.00 -> 134.9 mm, vias 0 -> 9
- net +5V: track 0.00 -> 120.0 mm, vias 0 -> 6
- net /CAN_RX: track 0.00 -> 39.1 mm
- net /CAN_TX: track 0.00 -> 35.2 mm
- net /USB_D-: track 0.00 -> 30.2 mm
- net /USB_D+: track 0.00 -> 30.0 mm
- net /SD_MISO: track 0.00 -> 24.5 mm, vias 0 -> 1
- net /SD_CS: track 0.00 -> 22.8 mm, vias 0 -> 1
- net /SD_MOSI: track 0.00 -> 21.7 mm, vias 0 -> 1
- net /RS485_RX: track 0.00 -> 21.1 mm, vias 0 -> 1
- net /RS485_TX: track 0.00 -> 20.1 mm, vias 0 -> 1
- net /RS485_DE: track 0.00 -> 16.3 mm, vias 0 -> 1
- net Net-(U4-CLK): track 0.00 -> 15.7 mm
- net /GPIO3: track 0.00 -> 15.2 mm, vias 0 -> 1
- net /CANH: track 0.00 -> 14.1 mm
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- added copper zone on B.Cu, net GND
- added copper zone on F.Cu, net GND
- added copper zone on In1.Cu, net GND
- added copper zone on In2.Cu, net GND
Other:
- copper layers 2 -> 4
