File: KleverLogger.kicad_sch (KiCad schematic)
At the start: 50 parts, among them J1 CAN, J5 USB_C_Receptacle_USB2.0, J7 RS485, U1 ESP32-C3-WROOM-02, U2 AP2112K-3.3, U3 TJA1051T-3, U5 MAX485E, U6 USBLC6-2SC6, U9 LM5164DDA

Commit message: USB updates
Parts:
- added C8: 100n, Capacitor_SMD:C_0805_2012Metric, symbol Device:C
- added J2: BATTERY, Connector_JST:JST_PH_S2B-PH-K_1x02_P2.00mm_Horizontal, symbol Connector_Generic:Conn_01x02
Connections:
- net +5V: now also U6.5 (VBUS), C8.1
- net GND: now also C8.2, J2.2 (Pin_2)
- net USB_D+: now also U6.4 (I/O2)
- net USB_D-: now also U6.6 (I/O1)
- net Vbus: now also J5.A4 (VBUS), J5.A9 (VBUS), J5.B4 (VBUS), J5.B9 (VBUS)
- net at U6.1 (I/O1): now also J5.A6 (D+), J5.B6 (D+)
- net at U6.3 (I/O2): now also J5.A7 (D-), J5.B7 (D-)
- net BAT+ renamed VIN
- net C3_DE_RS485 renamed RS485_DE
- net C3_RX renamed RS485_RX
- net C3_TX renamed RS485_TX
- no-connect marks 4 -> 3
Other:
- moved on the sheet: C35, C36, C37, C50, C52, C53, D5, L2, R67, R83, R84, R85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

Commit message: Update to components
Parts:
- added C9: C, symbol Device:C
Connections:
- net +3V3: now also C9.1
- net GND: now also C9.2
- net GPIO10: now reaches U1.10 (IO10)
- net GPI019: now reaches U1.13 (IO18)
- net GPIO7: now reaches U1.6 (IO7)
Other:
- moved on the sheet: C35, C36, C37, C50, C52, C53, L2, R67, R83, R84, R85, U9

Commit message: After ordering v0.1
Parts:
- removed C1, C2: 10uF/6.3V, Capacitor_SMD:C_0805_2012Metric, symbol Fair:C_0402_10uF/6.3V
- removed C3: 1uF/25V, Capacitor_SMD:C_0805_2012Metric, symbol Fair:C_0402_1uF/25V
- removed R2: 10k, Resistor_SMD:R_0805_2012Metric, symbol Fair:R_0402_10k
- removed S2: TL3340AF160QG, Fair:SW_TL3340AF160QG, symbol Fair:Switch_SMD_TL3340AF160QG
- added C1, C10, C11, C2, C3: 100n, Capacitor_SMD:C_0805_2012Metric, symbol Device:C
- added C12, C13: 10u, Capacitor_SMD:C_0805_2012Metric, symbol Device:C
- added D3, D4: 100V/3A, Diode_SMD:D_SOD-123F, symbol Device:D_Schottky
- added D6, D7, D8: WS2812B, LED_SMD:LED_WS2812B_PLCC4_5.0x5.0mm_P3.2mm, symbol LED:WS2812B
- added R17: 10, Resistor_SMD:R_0805_2012Metric, symbol Device:R
- added R2: 10k, Resistor_SMD:R_0805_2012Metric, symbol Fair_R_0805:10k
- added SW1: SW_SPST, Fair:Flat_SMD_Switch, symbol Switch:SW_SPST
- added TP1: 3V3, Fair:TestPoint_Pad_D0.8mm, symbol Connector:TestPoint_Small
- added TP10: CANH, Fair:TestPoint_Pad_D0.8mm, symbol Connector:TestPoint_Small
- added TP11: CANL, Fair:TestPoint_Pad_D0.8mm, symbol Connector:TestPoint_Small
- added TP12: IO3, Fair:TestPoint_Pad_D0.8mm, symbol Connector:TestPoint_Small
- added TP2: 5V, Fair:TestPoint_Pad_D0.8mm, symbol Connector:TestPoint_Small
- added TP3: RX, Fair:TestPoint_Pad_D0.8mm, symbol Connector:TestPoint_Small
- added TP4: DE, Fair:TestPoint_Pad_D0.8mm, symbol Connector:TestPoint_Small
- added TP5: TX, Fair:TestPoint_Pad_D0.8mm, symbol Connector:TestPoint_Small
- added TP6: MOSI, Fair:TestPoint_Pad_D0.8mm, symbol Connector:TestPoint_Small
- added TP7: MISO, Fair:TestPoint_Pad_D0.8mm, symbol Connector:TestPoint_Small
- added TP8: SCK, Fair:TestPoint_Pad_D0.8mm, symbol Connector:TestPoint_Small
- added TP9: CS, Fair:TestPoint_Pad_D0.8mm, symbol Connector:TestPoint_Small
- C35, C50: LCSC C1604 -> C28260
- C37: LCSC C14857 -> (none)
- C4: LCSC (none) -> C49678; Package (none) -> 0805
- C5: LCSC (none) -> C377773; Package (none) -> 0805
- C6, C7: value C -> 100n; footprint (none) -> Capacitor_SMD:C_0805_2012Metric; LCSC (none) -> C49678; Package (none) -> 0805
- C8: LCSC (none) -> C49678
- C9: value C -> 10u; footprint (none) -> Capacitor_SMD:C_0805_2012Metric; LCSC (none) -> C15850; Package (none) -> 0805
- R10: LCSC (none) -> C17437
- R11, R12, R13: LCSC (none) -> C17415; Package (none) -> 0805
- R67: LCSC C416833 -> (none)
- R83: LCSC C367975 -> (none)
- R84: LCSC C17719 -> (none)
Connections:
- net GPI019 is gone; now on net USB_D-: U1.13 (IO18)
- net GPIO10 is gone; now on net RS485_DE: U1.10 (IO10)
- net GPIO7 is gone; now on net SD_CS: U1.6 (IO7)
- net +3V3: now also C10.1, C13.1, C2.1, R2.2, TP1.1; no longer C6.1
- net +5V: now also C6.1, C1.1, C12.1, C3.1, D4.1 (K), D6.1 (VDD), D7.1 (VDD), D8.1 (VDD), TP2.1; no longer J1.4 (Pin_4)
- net BST: now also C50.2; no longer C50.1
- net CANH: now also J1.3 (Pin_3), TP10.1; no longer J1.2 (Pin_2)
- net CANL: now also J1.2 (Pin_2), TP11.1; no longer J1.3 (Pin_3)
- net EN/CHIP_PU: now also C11.1, R2.1
- net GND: now also J1.4 (Pin_4), C1.2, C10.2, C11.2, C12.2, C13.2, C2.2, C3.2, D6.3 (VSS), D7.3 (VSS), D8.3 (VSS), SW1.2 (B); no longer J1.1 (Pin_1)
- net RS485_DE: now also TP4.1; no longer U1.14 (IO19)
- net RS485_RX: now also TP3.1
- net RS485_TX: now also TP5.1
- net SD_CS: now also TP9.1
- net SD_MISO: now also TP7.1
- net SD_MOSI: now also TP6.1
- net SD_SCK: now also TP8.1
- net SW: now also C50.1; no longer C50.2
- net USB_D+: now also U1.14 (IO19)
- net VIN: now also D3.1 (K)
- net at D2.1 (A1), J7.3 (Pin_3): now also R11.2; no longer R12.2
- net at J5.A6 (D+), J5.B6 (D+): now also U6.3 (I/O2); no longer U6.1 (I/O1)
- net at J5.A7 (D-), J5.B7 (D-): now also U6.1 (I/O1); no longer U6.3 (I/O2)
- net at D2.2 (A2), J7.1 (Pin_1): now also R12.2; no longer R11.2
- net at J2.1 (Pin_1): now also D3.2 (A)
- net GPIO3: now reaches U1.15 (IO3)
- net GPIO3: now also R17.1, TP12.1
- net at U1.8 (IO9): now also SW1.1 (A)
- net LED_Green renamed GPIO2
- new net: D4.2 (A), J1.1 (Pin_1)
- new net: D7.2 (DOUT), D8.4 (DIN)
- new net: D6.2 (DOUT), D7.4 (DIN)
- new net: D6.4 (DIN), R17.2
- no-connect marks 3 -> 4
Other:
- moved on the sheet: C50, C8, D5, H1, H2, J5, R8, R9, U6
